Commit message: feat: implemented two types of mid360 emulation and enables automatic switching.

File: moudles/mecanum_car/robot.urdf (robot description, URDF)
Before this commit: robot mecanum_robot, 13 links, 12 joints
Links:
- added link base_link
Joints:
- added joint base_link_to_body: type fixed, parent base_link, child body, origin xyz=0 0 0 rpy=0 0 0
- joint front_left_wheel_joint: axis 0 0 1 -> 0 1 0; origin xyz=0.25 0.25 -0.075 rpy=1.5707 0 0 -> xyz=0.25 0.25 -0.075 rpy=0 0 0
- joint front_right_wheel_joint: axis 0 0 1 -> 0 1 0; origin xyz=0.25 -0.25 -0.075 rpy=1.5707 0 0 -> xyz=0.25 -0.25 -0.075 rpy=0 0 0
- joint rear_left_wheel_joint: axis 0 0 1 -> 0 1 0; origin xyz=-0.25 0.25 -0.075 rpy=1.5707 0 0 -> xyz=-0.25 0.25 -0.075 rpy=0 0 0
- joint rear_right_wheel_joint: axis 0 0 1 -> 0 1 0; origin xyz=-0.25 -0.25 -0.075 rpy=1.5707 0 0 -> xyz=-0.25 -0.25 -0.075 rpy=0 0 0

Commit message: feat: add lidar mode switching and fix mecanum wheel configuration
- Add sim_config.yaml for configuring lidar simulation mode (rgl/gpu_lidar/auto)
- Support automatic detection of NVIDIA GPU and fallback to gpu_lidar
- Fix mecanum wheel friction direction using gz:expressed_in attribute
- Update wheel pose to rpy=-1.5707 and fdir1 configuration per official example
- Add xmlns:gz namespace for Gazebo schema support
- Update README with lidar mode documentation

File: moudles/mecanum_car/robot.urdf (robot description, URDF)
Before this commit: robot mecanum_robot, 14 links, 13 joints
Joints:
- joint front_left_wheel_joint: axis 0 1 0 -> 0 0 1; origin xyz=0.25 0.25 -0.075 rpy=0 0 0 -> xyz=0.25 0.25 -0.075 rpy=1.5707 0 0
- joint front_right_wheel_joint: axis 0 1 0 -> 0 0 1; origin xyz=0.25 -0.25 -0.075 rpy=0 0 0 -> xyz=0.25 0.25 -0.075 rpy=1.5707 0 0
- joint rear_left_wheel_joint: axis 0 1 0 -> 0 0 1; origin xyz=-0.25 0.25 -0.075 rpy=0 0 0 -> xyz=-0.25 0.25 -0.075 rpy=1.5707 0 0
- joint rear_right_wheel_joint: axis 0 1 0 -> 0 0 1; origin xyz=-0.25 -0.25 -0.075 rpy=0 0 0 -> xyz=-0.25 -0.25 -0.075 rpy=1.5707 0 0
