Commit message: refactor: normalize simulation package layout

File: models/mecanum_car/robot.urdf (robot description, URDF)
Before this commit: robot mecanum_robot, 14 links, 13 joints
Joints:
- joint front_right_wheel_joint: origin xyz=0.25 0.25 -0.075 rpy=1.5707 0 0 -> xyz=0.25 -0.25 -0.075 rpy=1.5707 0 0

Commit message: refactor: rebuild mecanum car model following rmoss conventions
- Fix wheel detachment by correcting positions (Y ±0.25 → ±0.21) and
  collision radius (0.15m → 0.076m) to match DAE mesh dimensions
- Fix robot floating by moving chassis origin to wheel axle level (Z=0)
  and adjusting spawn height (0.28 → 0.1)
- Replace horizontal light bar with two vertical strips per armor plate,
  increase armor height from 55mm to 125mm (rmoss rm21_armor_module style)
- Add chassis IMU sensor (200Hz) and corresponding ros_gz_bridge
- Add missing Gazebo GUI plugins (GzSceneManager, InteractiveViewControl)
- Add DAE mesh assets for chassis, wheels, and gimbal

File: models/mecanum_car/robot.urdf (robot description, URDF)
Before this commit: robot mecanum_robot, 14 links, 13 joints
Links:
- removed link gimbal_base
- removed link gimbal_pitch_bracket
- added link armor_front; visual box size=0.012 0.135 0.125
- added link armor_left; visual box size=0.135 0.012 0.125
- added link armor_rear; visual box size=0.012 0.135 0.125
- added link armor_right; visual box size=0.135 0.012 0.125
- link chassis: geometry visual mesh filename=package://rm_sim_26/models/mecanum_car/meshes/chassis_base.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
- link front_left_wheel_link: geometry visual mesh filename=package://rm_sim_26/models/mecanum_car/meshes/wheel_left.dae
- link front_right_wheel_link: geometry visual mesh filename=package://rm_sim_26/models/mecanum_car/meshes/wheel_right.d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
- link gimbal_pitch: geometry visual mesh filename=package://rm_sim_26/models/mecanum_car/meshes/gimbal_pitch.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
- link gimbal_yaw: geometry visual mesh filename=package://rm_sim_26/models/mecanum_car/meshes/gimbal_yaw.dae
- link rear_left_wheel_link: geometry visual mesh filename=package://rm_sim_26/models/mecanum_car/meshes/wheel_right.d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
- link rear_right_wheel_link: geometry visual mesh filename=package://rm_sim_26/models/mecanum_car/meshes/wheel_left.dae
Joints:
- removed joint gimbal_base_joint
- removed joint gimbal_pitch_bracket_joint
- added joint armor_front_joint: type fixed, parent chassis, child armor_front, origin xyz=0.243 0 0.10 rpy=0 0 0
- added joint armor_left_joint: type fixed, parent chassis, child armor_left, origin xyz=0 0.184 0.10 rpy=0 0 0
- added joint armor_rear_joint: type fixed, parent chassis, child armor_rear, origin xyz=-0.243 0 0.10 rpy=0 0 0
- added joint armor_right_joint: type fixed, parent chassis, child armor_right, origin xyz=0 -0.184 0.10 rpy=0 0 0
- joint body_to_chassis: origin xyz=0 0 0.225 rpy=0 0 0 -> xyz=0 0 0 rpy=0 0 0
- joint front_left_wheel_joint: axis 0 0 1 -> 0 1 0; origin xyz=0.25 0.25 -0.075 rpy=1.5707 0 0 -> xyz=0.20 0.21 0 rpy=0 0 0
- joint front_right_wheel_joint: axis 0 0 1 -> 0 1 0; origin xyz=0.25 -0.25 -0.075 rpy=1.5707 0 0 -> xyz=0.20 -0.21 0 rpy=0 0 0
- joint gimbal_pitch_joint: origin xyz=0.06 0 0 rpy=0 0 0 -> xyz=0.06 0 0.08 rpy=0 0 0; parent gimbal_pitch_bracket -> gimbal_yaw
- joint gimbal_yaw_joint: origin xyz=0 0 0.08 rpy=0 0 0 -> xyz=0 0 0.205 rpy=0 0 0; parent gimbal_base -> chassis
- joint imu_joint: origin xyz=0 0 0 rpy=0 0 0 -> xyz=0 0 0.12 rpy=0 0 0
- joint lidar_joint: origin xyz=0.2 0 0.125 rpy=0 0 0 -> xyz=0.20 0 0.253 rpy=0 0 0
- joint rear_left_wheel_joint: axis 0 0 1 -> 0 1 0; origin xyz=-0.25 0.25 -0.075 rpy=1.5707 0 0 -> xyz=-0.20 0.21 0 rpy=0 0 0
- joint rear_right_wheel_joint: axis 0 0 1 -> 0 1 0; origin xyz=-0.25 -0.25 -0.075 rpy=1.5707 0 0 -> xyz=-0.20 -0.21 0 rpy=0 0 0
